File: SKINNY_PROTOTYPE/BB_Hardware/PCB/BadukBot/BotSchematic/_autosave-BotSchematic.kicad_pcb (KiCad board)
At the start: 2 copper layers, 68 parts, among them J1 MOLEX_78171-0002, J2 MOLEX_78171-0003, Q1 MMBT3904LT1G, Q2 MMBT3904LT1G, Q3 MMBT3904LT1G, Q4 MMBT3904LT1G, U1 STM32F051C8U6, U2 LSM6DS3, U3 A3901SEJTR-T, U4 ADP122ACPZ-3.3-R7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

Commit message: PCB adjustments
Parts:
- moved C13 3.30 mm to (229.4, 74.8), turned to 270 degrees
- moved U5 1.95 mm to (219.2, 75.3)
- moved U4 1.78 mm to (226.4, 74.8)
- moved C14 1.38 mm to (218.7, 70.8)
- moved R15 1.38 mm to (216.5, 71.3)
- moved C12 0.91 mm to (224.3, 74.8)
- moved J2 0.90 mm to (218.2, 84.1)
- moved R14 0.90 mm to (216.9, 79.5)
- moved R19 0.90 mm to (218.1, 79.5)
- moved R20 0.90 mm to (219.3, 79.5)
Other:
- copper layers 2 -> 4
Changed lines of the file:
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@@
   (general
     (thickness 1.6)
-    (drawings 13)
+    (drawings 17)
     (tracks 0)
     (zones 0)
@@
   (layers
     (0 F.Cu signal)
+    (1 In1.Cu signal)
+    (2 In2.Cu signal)
     (31 B.Cu signal)
-    (32 B.Adhes user)
     (33 F.Adhes user)
-    (34 B.Paste user)
     (35 F.Paste user)
-    (36 B.SilkS user)
     (37 F.SilkS user)
-    (38 B.Mask user)
     (39 F.Mask user)
     (40 Dwgs.User user)
@@
     (46 B.CrtYd user)
     (47 F.CrtYd user)
-    (48 B.Fab user)
     (49 F.Fab user)
   )
@@
   )
   (module AT42QT1070-MMHCT-ND:VQFN_20PAD (layer F.Cu)
-    (at 217.251874 75.165421 90)
+    (at 219.2 75.3 90)
     (attr smd)
     (fp_text reference U5 (at -1.85 -1.7 90) (layer F.SilkS)
@@
   )
   (module 1uF:0603ZD105KAT2A (layer F.Cu)
-    (at 225.2 74.95 90)
+    (at 224.3 74.85 90)
     (fp_text reference C12 (at 0.05 1.4 90) (layer F.SilkS)
       (effects (font (size 0.5 0.5) (thickness 0.125)))
@@
   )
   (module 1uF:0603ZD105KAT2A (layer F.Cu)
-    (at 228.116518 71.827084 180)
-    (fp_text reference C13 (at -0.109066 1.444024 180) (layer F.SilkS)
-      (effects (font (size 0.5 0.5) (thickness 0.125)))
-    )
-    (fp_text value 1uF (at 0 0 180) (layer F.SilkS)
+    (at 229.45 74.85 270)
+    (fp_text reference C13 (at -0.109066 1.444024 270) (layer F.SilkS)
+      (effects (font (size 0.5 0.5) (thickness 0.125)))
+    )
+    (fp_text value 1uF (at 0 0 270) (layer F.SilkS)
       (effects (font (size 1 1) (thickness 0.15)))
     )
@@
     (fp_line (start -0.3683 -0.4826) (end -0.8763 -0.4826) (layer F.Fab) (width 0.1524))
     (fp_line (start -0.3683 0.4826) (end -0.3683 -0.4826) (layer F.Fab) (width 0.1524))
-    (fp_text user * (at 0 0 180) (layer F.Fab)
-      (effects (font (size 1 1) (thickness 0.15)))
-    )
-    (fp_text user * (at 0 0 180) (layer F.SilkS)
-      (effects (font (size 1 1) (thickness 0.15)))
-    )
-    (fp_text user "Copyright 2016 Accelerated Designs. All rights reserved." (at 0 0 180) (layer Cmts.User)
-      (effects (font (size 0.127 0.127) (thickness 0.002)))
-    )
-    (pad 2 smd rect (at 0.7239 0 180) (size 0.7112 0.9652) (layers F.Cu F.Paste F.Mask)
-      (net 4 GND))
-    (pad 1 smd rect (at -0.7239 0 180) (size 0.7112 0.9652) (layers F.Cu F.Paste F.Mask)
+    (fp_text user * (at 0 0 270) (layer F.Fab)
+      (effects (font (size 1 1) (thickness 0.15)))
+    )
+    (fp_text user * (at 0 0 270) (layer F.SilkS)
+      (effects (font (size 1 1) (thickness 0.15)))
+    )
+    (fp_text user "Copyright 2016 Accelerated Designs. All rights reserved." (at 0 0 270) (layer Cmts.User)
+      (effects (font (size 0.127 0.127) (thickness 0.002)))
+    )
+    (pad 2 smd rect (at 0.7239 0 270) (size 0.7112 0.9652) (layers F.Cu F.Paste F.Mask)
+      (net 4 GND))
+    (pad 1 smd rect (at -0.7239 0 270) (size 0.7112 0.9652) (layers F.Cu F.Paste F.Mask)
       (net 9 +3V3))
   )
@@
   )
   (module MOLEX_78171-0003:MOLEX_78171-0003_0 (layer F.Cu)
-    (at 217.251874 84.115421)
+    (at 218.151874 84.115421)
     (descr "Pico-EZmate Wire-to-Board Header, Vertical, Housing Height 1.55mm, with Side Friction Locks, 3 Circuits")
     (attr smd)
@@
   )
   (module ADP122ACPZ-3.3-R7:SON65P200X200X60-7N-D (layer F.Cu)
-    (at 228.216518 75.077084 270)
+    (at 226.45 74.85 270)
     (descr CP-6-3)
     (tags "Integrated Circuit")
@@
   )
   (module 100nf:C0402C104K4RACTU (layer F.Cu)
-    (at 217.751874 71.815421)
+    (at 218.651874 70.765421)
     (fp_text reference C14 (at 0 -0.9) (layer F.SilkS)
       (effects (font (size 0.5 0.5) (thickness 0.125)))
@@
   )
   (module 10K0402:CRCW040210K0FKED (layer F.Cu)
-    (at 216.048561 79.546356 270)
+    (at 216.948561 79.546356 270)
     (fp_text reference R14 (at 0 0.9 270) (layer F.SilkS)
       (effects (font (size 0.5 0.5) (thickness 0.125)))
@@
   )
   (module 100K:CRCW0402100KFKED (layer F.Cu)
-    (at 215.551874 72.315421 90)
+    (at 216.451874 71.265421 90)
     (fp_text reference R15 (at 0 -0.95 90) (layer F.SilkS)
       (effects (font (size 0.5 0.5) (thickness 0.125)))
@@
   )
   (module 10K0402:CRCW040210K0FKED (layer F.Cu)
-    (at 217.248561 79.546356 270)
+    (at 218.148561 79.546356 270)
     (fp_text reference R19 (at -1.75 -0.65 270) (layer F.SilkS)
       (effects (font (size 0.5 0.5) (thickness 0.125)))
@@
   )
   (module 10K0402:CRCW040210K0FKED (layer F.Cu)
-    (at 218.448561 79.546356 270)
+    (at 219.348561 79.546356 270)
     (fp_text reference R20 (at 0 -0.95 270) (layer F.SilkS)
       (effects (font (size 0.5 0.5) (thickness 0.125)))
@@
       (net 9 +3V3))
   )
-  (gr_line (start 208.1 154.25) (end 208.05 65.7) (layer F.SilkS) (width 0.2))
-  (gr_line (start 235.45 154.3) (end 208.1 154.25) (layer F.SilkS) (width 0.2))
-  (gr_line (start 235.45 65.65) (end 235.45 154.3) (layer F.SilkS) (width 0.2))
-  (gr_line (start 208.05 65.7) (end 235.45 65.65) (layer F.SilkS) (width 0.2))
+  (gr_line (start 204.75 105.25) (end 188.75 105.25) (layer F.SilkS) (width 0.2))
+  (gr_line (start 188.75 111.8) (end 204.75 111.8) (layer F.SilkS) (width 0.2))
+  (gr_line (start 188.75 111.75) (end 188.75 105.25) (layer F.SilkS) (width 0.2))
+  (gr_line (start 204.75 105.25) (end 204.75 111.8) (layer F.SilkS) (width 0.2))
+  (gr_line (start 212.75 149.8) (end 212.75 69.5) (layer F.SilkS) (width 0.2))
+  (gr_line (start 231.85 149.8) (end 212.8 149.8) (layer F.SilkS) (width 0.2))
+  (gr_line (start 231.8 69.5) (end 231.85 149.85) (layer F.SilkS) (width 0.2))
+  (gr_line (start 212.75 69.5) (end 231.8 69.5) (layer F.SilkS) (width 0.2))
   (gr_circle (center 222.35 109.7) (end 217.2 116.8) (layer F.SilkS) (width 0.2))
   (gr_line (start 213.4 149.45) (end 213.35 120.25) (layer F.SilkS) (width 0.2))
