File: SKINNY_PROTOTYPE/BB_Hardware/PCB/BadukBot/BotSchematic/offset.kicad_pcb (KiCad board)
At the start: 4 copper layers, 22.4 x 87.6 mm, 72 parts, among them J1 MOLEX_78171-0002, J10 A3-16DA-2SV(71), J11 62401621722, J12 803-87-010-10-001101, J13 67997-410HLF, J2 MOLEX_78171-0003, Q1 MMBT3904LT1G, Q2 MMBT3904LT1G, Q3 MMBT3904LT1G, Q4 MMBT3904LT1G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

Commit message: Original board layer images added; Experiments with trace routing using FreeRouting and component placement in KiCAD
Parts:
- moved U7 0.92 mm to (217.2, 139.8), turned to 180 degrees
Other:
- net class Default: clearance 0.2 -> 0.127; trace_width 0.25 -> 0.1524; via_dia 0.8 -> 0.254; via_drill 0.4 -> 0.1016
- rule pad_to_mask_clearance: 0.2 -> 0.0508
- rule trace_clearance: 0.2 -> 0.127
- rule trace_min: 0.2 -> 0.127
- rule via_min_drill: 0.3 -> 0.0508
- rule via_min_size: 0.4 -> 0.254
Changed lines of the file:
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@@
   )
   (setup
-    (last_trace_width 0.25)
-    (trace_clearance 0.2)
+    (last_trace_width 0.1524)
+    (trace_clearance 0.127)
     (zone_clearance 0.508)
     (zone_45_only no)
-    (trace_min 0.2)
+    (trace_min 0.127)
     (segment_width 0.2)
     (edge_width 0.15)
-    (via_size 0.8)
-    (via_drill 0.4)
-    (via_min_size 0.4)
-    (via_min_drill 0.3)
+    (via_size 0.254)
+    (via_drill 0.1016)
+    (via_min_size 0.254)
+    (via_min_drill 0.0508)
     (uvia_size 0.3)
     (uvia_drill 0.1)
@@
     (pad_size 1.524 1.524)
     (pad_drill 0.762)
-    (pad_to_mask_clearance 0.2)
+    (pad_to_mask_clearance 0.0508)
     (aux_axis_origin 0 0)
-    (visible_elements FFFDFF7F)
+    (visible_elements FFFDF77F)
     (pcbplotparams
       (layerselection 0x010fc_ffffffff)
@@
   (net 124 15b_GND2)
   (net_class Default "This is the default net class."
-    (clearance 0.2)
-    (trace_width 0.25)
-    (via_dia 0.8)
-    (via_drill 0.4)
+    (clearance 0.127)
+    (trace_width 0.1524)
+    (via_dia 0.254)
+    (via_drill 0.1016)
     (uvia_dia 0.3)
     (uvia_drill 0.1)
@@
   )
   (module digikey-footprints:QFN-20-1EP_4x4mm_RevA (layer F.Cu)
-    (at 216.65 139.15 145)
-    (fp_text reference U7 (at 2.218104 2.014499 145) (layer F.SilkS)
-      (effects (font (size 0.5 0.5) (thickness 0.125)))
-    )
-    (fp_text value NRF24L01P-R7 (at 0 2.9 145) (layer F.Fab)
+    (at 217.25 139.85 180)
+    (fp_text reference U7 (at 2.218104 2.014499 180) (layer F.SilkS)
+      (effects (font (size 0.5 0.5) (thickness 0.125)))
+    )
+    (fp_text value NRF24L01P-R7 (at 0 2.9 180) (layer F.Fab)
       (effects (font (size 1 1) (thickness 0.15)))
     )
@@
     (fp_line (start 1.8 -1.8) (end 1.8 -1.1) (layer F.SilkS) (width 0.1))
     (fp_line (start -1.5 1.5) (end 1.5 1.5) (layer F.Fab) (width 0.1))
-    (fp_text user REF** (at 0 0 145) (layer F.Fab)
+    (fp_text user REF** (at 0 0 180) (layer F.Fab)
       (effects (font (size 0.5 0.5) (thickness 0.05)))
     )
     (fp_line (start 1.5 -1.5) (end 1.5 1.5) (layer F.Fab) (width 0.1))
-    (pad 16 smd rect (at 1 -1.7 145) (size 0.25 0.4) (layers F.Cu F.Paste F.Mask)
+    (pad 16 smd rect (at 1 -1.7 180) (size 0.25 0.4) (layers F.Cu F.Paste F.Mask)
       (net 28 "Net-(R27-Pad2)"))
-    (pad 17 smd rect (at 0.5 -1.7 145) (size 0.25 0.4) (layers F.Cu F.Paste F.Mask)
+    (pad 17 smd rect (at 0.5 -1.7 180) (size 0.25 0.4) (layers F.Cu F.Paste F.Mask)
       (net 124 15b_GND2))
-    (pad 18 smd rect (at 0 -1.7 145) (size 0.25 0.4) (layers F.Cu F.Paste F.Mask)
+    (pad 18 smd rect (at 0 -1.7 180) (size 0.25 0.4) (layers F.Cu F.Paste F.Mask)
       (net 123 1b_3.3v))
-    (pad 19 smd rect (at -0.5 -1.7 145) (size 0.25 0.4) (layers F.Cu F.Paste F.Mask)
+    (pad 19 smd rect (at -0.5 -1.7 180) (size 0.25 0.4) (layers F.Cu F.Paste F.Mask)
       (net 7 "Net-(C22-Pad1)"))
-    (pad 20 smd rect (at -1 -1.7 145) (size 0.25 0.4) (layers F.Cu F.Paste F.Mask)
+    (pad 20 smd rect (at -1 -1.7 180) (size 0.25 0.4) (layers F.Cu F.Paste F.Mask)
       (net 124 15b_GND2))
-    (pad 10 smd rect (at 1 1.7 145) (size 0.25 0.4) (layers F.Cu F.Paste F.Mask)
+    (pad 10 smd rect (at 1 1.7 180) (size 0.25 0.4) (layers F.Cu F.Paste F.Mask)
       (net 44 RADIO_CLK))
-    (pad 9 smd rect (at 0.5 1.7 145) (size 0.25 0.4) (layers F.Cu F.Paste F.Mask)
+    (pad 9 smd rect (at 0.5 1.7 180) (size 0.25 0.4) (layers F.Cu F.Paste F.Mask)
       (net 60 "Net-(U7-Pad9)"))
-    (pad 8 smd rect (at 0 1.7 145) (size 0.25 0.4) (layers F.Cu F.Paste F.Mask)
+    (pad 8 smd rect (at 0 1.7 180) (size 0.25 0.4) (layers F.Cu F.Paste F.Mask)
       (net 124 15b_GND2))
-    (pad 7 smd rect (at -0.5 1.7 145) (size 0.25 0.4) (layers F.Cu F.Paste F.Mask)
+    (pad 7 smd rect (at -0.5 1.7 180) (size 0.25 0.4) (layers F.Cu F.Paste F.Mask)
       (net 123 1b_3.3v))
-    (pad 6 smd rect (at -1 1.7 145) (size 0.25 0.4) (layers F.Cu F.Paste F.Mask)
+    (pad 6 smd rect (at -1 1.7 180) (size 0.25 0.4) (layers F.Cu F.Paste F.Mask)
       (net 48 RADIO_IRQ))
-    (pad 11 smd rect (at 1.7 1 145) (size 0.4 0.25) (layers F.Cu F.Paste F.Mask)
+    (pad 11 smd rect (at 1.7 1 180) (size 0.4 0.25) (layers F.Cu F.Paste F.Mask)
       (net 97 14b_VDD_PA))
-    (pad 12 smd rect (at 1.7 0.5 145) (size 0.4 0.25) (layers F.Cu F.Paste F.Mask)
+    (pad 12 smd rect (at 1.7 0.5 180) (size 0.4 0.25) (layers F.Cu F.Paste F.Mask)
       (net 99 12b_ANT1))
-    (pad 13 smd rect (at 1.7 0 145) (size 0.4 0.25) (layers F.Cu F.Paste F.Mask)
+    (pad 13 smd rect (at 1.7 0 180) (size 0.4 0.25) (layers F.Cu F.Paste F.Mask)
       (net 98 13b_ANT2))
-    (pad 14 smd rect (at 1.7 -0.5 145) (size 0.4 0.25) (layers F.Cu F.Paste F.Mask)
+    (pad 14 smd rect (at 1.7 -0.5 180) (size 0.4 0.25) (layers F.Cu F.Paste F.Mask)
       (net 124 15b_GND2))
-    (pad 15 smd rect (at 1.7 -1 145) (size 0.4 0.25) (layers F.Cu F.Paste F.Mask)
+    (pad 15 smd rect (at 1.7 -1 180) (size 0.4 0.25) (layers F.Cu F.Paste F.Mask)
       (net 123 1b_3.3v))
-    (pad 5 smd rect (at -1.7 1 145) (size 0.4 0.25) (layers F.Cu F.Paste F.Mask)
+    (pad 5 smd rect (at -1.7 1 180) (size 0.4 0.25) (layers F.Cu F.Paste F.Mask)
       (net 39 MISO))
-    (pad 4 smd rect (at -1.7 0.5 145) (size 0.4 0.25) (layers F.Cu F.Paste F.Mask)
+    (pad 4 smd rect (at -1.7 0.5 180) (size 0.4 0.25) (layers F.Cu F.Paste F.Mask)
       (net 40 MOSI))
-    (pad 3 smd rect (at -1.7 0 145) (size 0.4 0.25) (layers F.Cu F.Paste F.Mask)
+    (pad 3 smd rect (at -1.7 0 180) (size 0.4 0.25) (layers F.Cu F.Paste F.Mask)
       (net 38 SCK))
-    (pad 2 smd rect (at -1.7 -0.5 145) (size 0.4 0.25) (layers F.Cu F.Paste F.Mask)
+    (pad 2 smd rect (at -1.7 -0.5 180) (size 0.4 0.25) (layers F.Cu F.Paste F.Mask)
       (net 37 CSN))
-    (pad 21 smd rect (at 0 0 145) (size 2.6 2.6) (layers F.Cu F.Paste F.Mask)
+    (pad 21 smd rect (at 0 0 180) (size 2.6 2.6) (layers F.Cu F.Paste F.Mask)
       (net 124 15b_GND2))
-    (pad 1 smd rect (at -1.7 -1 145) (size 0.4 0.25) (layers F.Cu F.Paste F.Mask)
+    (pad 1 smd rect (at -1.7 -1 180) (size 0.4 0.25) (layers F.Cu F.Paste F.Mask)
       (net 41 RADIO_CE))
   )
