File: SKINNY_PROTOTYPE/BB_Hardware/PCB/BadukBot/BotSchematic/BotSchematic.sch (KiCad schematic (older format))
At the start: 1 part

Commit message: Converting Altium Schematic pdf to KiCAD Schematic
Parts:
- removed U?: LM1875T_NOPB, digikey-footprints:TO-220-5, symbol dk_Linear-Amplifiers-Audio:LM1875T_NOPB
- added ANT?: Antenna, digikey-footprints:Antenna_1.6x3.2mm_2450AT18A100E, symbol dk_RF-Antennas:2450AT18A100E
- added B1: nrf24l01, JOHANSON_2450BM14A0002T_0, symbol JOHANSON_2450BM14A0002T:JOHANSON_2450BM14A0002T
- added C1: 10nF, CC0402N, symbol 10nF:C0402C103J3RACTU
- added C10, C11, C4, C5, C6: 100nF, CC0402N, symbol 100nf:C0402C104K4RACTU
- added C12, C13, C2: 1uF, 0603, symbol 1uF:0603ZD105KAT2A
- added C15, C3: TAIYO_YUDEN_LMK107BJ475KA-T, TAIYO_YUDEN_LMK107BJ475KA-T_0, symbol TAIYO_YUDEN_LMK107BJ475KA-T:TAIYO_YUDEN_LMK107BJ475KA-T
- added C16: Taiyo, TAIYO_YUDEN_LMK107BJ475KA-T_0, symbol TAIYO_YUDEN_LMK107BJ475KA-T:TAIYO_YUDEN_LMK107BJ475KA-T
- added C21: 2.2nF, CC0402N, symbol 2.2nF_X7R_50V:C0402C222K5RACTU
- added C7, C8: 22pF, CAPC1005X55N, symbol 22pf_GRM1555C1H220JA01D:GRM1555C1H220JA01D
- added D1, D3: PD15-22C_TR8, digikey-footprints:SMD-4_3.3x2.8_PD15-22C_TR8, symbol dk_Optical-Sensors-Photodiodes:PD15-22C_TR8
- added D2: SMLVN6RGB1W1, LED310X280X60-6N, symbol SMLVN6RGB1W1:SMLVN6RGB1W1
- added J?: MOLEX_78171-0002, MOLEX_78171-0002_0, symbol MOLEX_78171-0002:MOLEX_78171-0002
- added P1: SWD Pads, symbol Connector_Generic:Conn_01x06
- added P4: Conn_01x02_Female, symbol Connector:Conn_01x02_Female
- added P5: Pads, symbol Connector:Conn_01x06_Female
- added Q1, Q2, Q3, Q4: MMBT3904LT1G, digikey-footprints:SOT-23-3, symbol dk_Transistors-Bipolar-BJT-Single:MMBT3904LT1G
- added R1, R2, R3: VISHAY_CRCW040222R0FKED, VISHAY_CRCW040222R0FKED_0, symbol 22r:VISHAY_CRCW040222R0FKED
- added R10, R13: 560K, RC0402N, symbol 560K:RC0402FR-07560KL
- added R11, R21: 1.5M, RES_CRCW_0402, symbol 1.5M:CRCW04021M50FKED
- added R12, R8: 100K, RES_CRCW_0402, symbol BotSchematic-cache:100K:CRCW0402100KFKED
- added R16: 22.6R, RC0402N, symbol 22_6R:ERJ-2RKF22R6X
- added R17: 130R, RC0402N, symbol 130R:ERJ-2RKF1300X
- added R18: 24.9R, RC0402N, symbol 24.9R:ERJ-2RKF24R9X
- added R22, R7, R9: 10K, RES_CRCW_0402, symbol 10K0402:CRCW040210K0FKED
- added R23, R4, R5, R6: 100K, RES_CRCW_0402, symbol 100K:CRCW0402100KFKED
- added R24: 0R, RC0402N, symbol symbols:ERJ-2GE0R00X
- added R25, R26: NC, symbol Device:R_US
- added U1: STM32F051C8U6, QFN50P700X700X65-49N-D, symbol STM32F051C8U6:STM32F051C8U6
- added U2: LSM6DS3, Package_LGA:LGA-14_3x2.5mm_P0.5mm_LayoutBorder3x4y, symbol Sensor_Motion:LSM6DS3
- added U4: ADP122ACPZ-3.3-R7, SON65P200X200X60-7N-D, symbol ADP122ACPZ-3.3-R7:ADP122ACPZ-3.3-R7
- added U6: MCP73831T-2ACI_OT, SOT-23-5_MC, symbol MCP:MCP73831T-2ACI_OT
- added Y1: 7V-16.000MAAE-T, OSCCC500X320X105N, symbol TXC-7V-16.000MAAE-T:7V-16.000MAAE-T
Connections:
- net labels added: +3.3V, +BATT, ANT1, ANT2, CHARGING, CSN, Charging, Earth, IMU_INT, IO1, IO2, MCU_X1_16MHZ, MCU_X2_16MHZ, MISO, MOSI, MOTOR_CONTROL1, MOTOR_CONTROL2, MOTOR_CONTROL3, MOTOR_CONTROL4, NRST, NSRT, PHOTODIODE_1, PHOTODIODE_2, RADIO_CE, RADIO_CLK, RADIO_IRQ, RGBLED1, RGBLED2, RGBLED3, SCK, SCL, SDA, SWCLK, SWDIO, TOUCH_CHG, VDD_PA
- wire segments 0 -> 159
Other:
- note added: "Antenna Circuit (Balun)"
- note added: "Charger"
- note added: "Crystal"
- note added: "Decoupling\nCapacitors"
- note added: "Ext Port"
- note added: "IMU"
- note added: "MCU"
- note added: "Orientation of crystal \ndoesn’t matter, works \nboth ways"
- note added: "Photodiodes"
- note added: "RGB LED"
- note added: "SWD\nConnector"
- note added: "VCC\nSWDIO\nnRESET\nSWCLK\nGND\nSWO"
- note added: "Voltage Regulator"

Commit message: Completed KiCAD Schematic
Parts:
- added C14, C17, C18, C19, C20: 100nF, CC0402N, symbol BotSchematic-cache:100nf:C0402C104K4RACTU
- added C22: 33nF, CAPC1005X55N, symbol 33nF:C1005X7R1H333K050BB
- added C9: 10uF, CAPC1608X9N, symbol 100uF:GRM188R61A106ME69D
- added J2: MOLEX_78171-0003, MOLEX_78171-0003_0, symbol MOLEX_78171-0003:MOLEX_78171-0003
- added P2, P3: Pad, symbol Connector:Conn_01x02_Female
- added R14, R19, R20: 10K, RES_CRCW_0402, symbol BotSchematic-cache:10K0402:CRCW040210K0FKED
- added R15: 100K, RES_CRCW_0402, symbol BotSchematic-cache:100K:CRCW0402100KFKED
- added R27: 22K, RESC1005X40N, symbol 22k:CRCW040222K0FKED
- added U5: AT42QT1070-MMHCT-ND, MODULE, symbol AT42QT1070-MMHCT-ND:AT42QT1070-MMHCT-ND
- added U7: NRF24L01P-R7, digikey-footprints:QFN-20-1EP_4x4mm_RevA, symbol dk_RF-Transceiver-ICs:NRF24L01P-R7
- added U?: A3901SEJTR-T, DFN300X300X75-11N, symbol A3901SEJTR-T:A3901SEJTR-T
Connections:
- net labels added: GND, ~TOUCH_CHG~
- net labels removed: Earth
- wire segments 159 -> 201
Other:
- note added: "Electrodes"
- note added: "Motor Controller"
- note added: "Radio Chip"
- note added: "Touch Sensing"
- note added: "Use 78172-0410 crimps\nUse with 78172-0003 housing"

Commit message: BOM updates; Converted Altium Schematics pdf to KiCAD; New PCB design; First pass at routing with FreeRouting
Parts:
- removed C9: 10uF, CAPC1608X9N, symbol 100uF:GRM188R61A106ME69D
- added C9: 10uF, 10uF:CAPC1608X9N, symbol 10uF:GRM188R61A106ME69D
- B1: footprint JOHANSON_2450BM14A0002T_0 -> JOHANSON_2450BM14A0002T:JOHANSON_2450BM14A0002T_0
- C1: footprint CC0402N -> 10nF:C0402C103J3RACTU
- C10, C11, C4, C5, C6: footprint CC0402N -> 100nf:C0402C104K4RACTU
- C12, C13, C2: footprint 0603 -> 1uF:0603ZD105KAT2A
- C14, C17, C18, C19, C20: footprint CC0402N -> 100nf:C0402C104K4RACTU; symbol BotSchematic-cache:100nf:C0402C104K4RACTU -> BotSchematic-rescue:100nf_C0402C104K4RACTU-BotSchematic-cache
- C15, C16, C3: footprint TAIYO_YUDEN_LMK107BJ475KA-T_0 -> TAIYO_YUDEN_LMK107BJ475KA-T:TAIYO_YUDEN_LMK107BJ475KA-T_0
- C21: footprint CC0402N -> 2.2nF X7R 50V:C0402C222K5RACTU
- C22: footprint CAPC1005X55N -> 33nF:CAPC1005X55N
- C7, C8: footprint CAPC1005X55N -> 22pf_GRM1555C1H220JA01D:CAPC1005X55N
- D2: footprint LED310X280X60-6N -> SMLVN6RGB1W1:LED310X280X60-6N
- J1: renamed from J?; footprint MOLEX_78171-0002_0 -> MOLEX_78171-0002:MOLEX_78171-0002_0
- J2: footprint MOLEX_78171-0003_0 -> MOLEX_78171-0003:MOLEX_78171-0003_0
- R1, R2, R3: footprint VISHAY_CRCW040222R0FKED_0 -> 22r:VISHAY_CRCW040222R0FKED_0
- R10, R13: footprint RC0402N -> 560K:RC0402FR-07560KL
- R11, R21: footprint RES_CRCW_0402 -> 1.5M:CRCW04021M50FKED
- R12, R15, R8: footprint RES_CRCW_0402 -> 100K:CRCW0402100KFKED; symbol BotSchematic-cache:100K:CRCW0402100KFKED -> BotSchematic-rescue:100K_CRCW0402100KFKED-BotSchematic-cache
- R14, R19, R20: footprint RES_CRCW_0402 -> 10K0402:CRCW040210K0FKED; symbol BotSchematic-cache:10K0402:CRCW040210K0FKED -> BotSchematic-rescue:10K0402_CRCW040210K0FKED-BotSchematic-cache
- R16: footprint RC0402N -> 22_6R:ERJ-2RKF22R6X
- R17: footprint RC0402N -> 130R:ERJ-2RKF1300X
- R18: footprint RC0402N -> 24.9R:ERJ-2RKF24R9X
- R22, R7, R9: footprint RES_CRCW_0402 -> 10K0402:CRCW040210K0FKED
- R23, R4, R5, R6: footprint RES_CRCW_0402 -> 100K:CRCW0402100KFKED
- R24: footprint RC0402N -> footprints:ERJ-2GE0R00X
- R25, R26: footprint (none) -> footprints:ERJ-2GE0R00X
- R27: footprint RESC1005X40N -> 22K:RESC1005X40N
- U1: footprint QFN50P700X700X65-49N-D -> STM32F051C8U6:QFN50P700X700X65-49N-D; Description (none) -> STM32F051C8U6
- U2: footprint Package_LGA:LGA-14_3x2.5mm_P0.5mm_LayoutBorder3x4y -> digikey-footprints:LGA-14L_2.5x3mm__LSM6DS3
- U3: renamed from U?; footprint DFN300X300X75-11N -> A3901SEJTR-T:DFN300X300X75-11N
- U4: footprint SON65P200X200X60-7N-D -> ADP122ACPZ-3.3-R7:SON65P200X200X60-7N-D
- U5: footprint MODULE -> AT42QT1070-MMHCT-ND:VQFN_20PAD
- U6: footprint SOT-23-5_MC -> MCP:MCP73831T-2ACI&slash_OT
- Y1: footprint OSCCC500X320X105N -> TXC-7V-16.000MAAE-T:OSCCC500X320X105N
- gave numbers to parts that had none: 1
Connections:
- no-connect marks 0 -> 35

Commit message: schematic/pcb changes
Parts:
- U5: footprint AT42QT1070-MMHCT-ND:VQFN_20PAD -> vq:VQFN_20PAD

Commit message: More work on the PCB
Parts:
- added J10: A3-16DA-2SV(71), A13:A13, symbol 16pos_2mm_SMD:A3-16DA-2SV(71)
- added J11: 62401621722, 16pos_2mm_RA:0877601616, symbol 16pos2mmRA:0877601616
- added J12: 803-87-010-10-001101, 2x5conn:2x5, symbol 2x5conn:67997-410HLF
- added J13: 67997-410HLF, 2x5conn:2x5, symbol 2x5conn:67997-410HLF
- added P20: charge pins, symbol Connector:Conn_01x02_Female
Connections:
- net labels added: 10a_SDA, 10b_SDA, 11a_SCL, 11b_SCL, 12a_ANT1, 12b_ANT1, 13a_ANT2, 13b_ANT2, 14a_VDD_PA, 14b_VDD_PA, 15a_GND2, 15a_P4-1, 15b_GND2, 15b_P4-1, 1a_3.3v, 1b_3.3v, 21a_3.3v, 21b_3.3v, 22a_VBAT, 22b_VBAT, 23a_GND, 23b_GND, 24a_IMU_INT, 24b_IMU_INT, 25a_SDA, 25b_SDA, 26a_SCL, 26b_SCL, 27a_CHARGING, 27b_CHARGING, 28a_P4-1, 2a_GND, 2b_GND, 3a_PHOTODIODE1, 3b_PHOTODIODE1, 4a_PHOTODIODE2, 4b_PHOTODIODE2, 5a_RGBLED1, 5b_RGBLED1, 6a_RGBLED2, 6b_RGBLED2, 7a_RGBLED3, 7b_RGBLED3, 8a_IO1, 8b_IO1, 9a_IO2, 9b_IO2, ~29a_TOUCH_CHG~, ~29b_TOUCH_CHG~
- net labels removed: +3.3V, +BATT, ANT1, ANT2, CHARGING, Charging, IMU_INT, IO1, IO2, PHOTODIODE_1, PHOTODIODE_2, RGBLED1, RGBLED2, RGBLED3, SCL, SDA, TOUCH_CHG, VDD_PA, ~TOUCH_CHG~
- wire segments 201 -> 374
Other:
- note added: "21a 3.3v\n22a VBAT\n23a GND\n24a IMU_INT\n25a SDA\n26a SCL\n27a CHARGING\n28a P4-1\n29a TOUCH_CHG\n30a P4"
- note added: "Pins to connections:\n1a 3.3v\n2a GND\n3a Photodiode1\n4a photodiode2\n5a RGBLED1\n6a RGBLED2\n7a RGBLED3\n8a IO1\n9a IO2\n10a SDA\n11a SCL\n12a ANT1\n13a ANT2\n14a VDD_PA\n15a P4-1\n16a_GND2\n"
- note added: "Pins to connections:\n1b 3.3v\n2b GND\n3b Photodiode1\n4b photodiode2\n5b RGBLED1\n6b RGBLED2\n7b RGBLED3\n8b IO1\n9b IO2\n10b SDA\n11b SCL\n12b ANT1\n13b ANT2\n14b VDD_PA\n15b P4-1\n\n21b 3.3v\n22b VBAT\n23b GND\n24b IMU_INT\n25b SDA\n26b SCL\n27b CHARGING\n28b P4-1\n29b TOUCH_CHG"
- moved on the sheet: C17, C18, C19, C20

Commit message: Images of original board's layers; images of current work setup; updated schematics and BOM to change connectors; major boards revisions
Parts:
- removed ANT1: Antenna, digikey-footprints:Antenna_1.6x3.2mm_2450AT18A100E, symbol dk_RF-Antennas:2450AT18A100E
- removed J12: 803-87-010-10-001101, 2x5conn:2x5, symbol 2x5conn:67997-410HLF
- removed J13: 67997-410HLF, 2x5conn:2x5, symbol 2x5conn:67997-410HLF
- removed P2, P3: Pad, symbol Connector:Conn_01x02_Female
- removed P20: charge pins, symbol Connector:Conn_01x02_Female
- added ANT1: 2450AT18D0100E, 2450AT18D0100E:DFN320X160X120-4RN, symbol 2450AT18D0100E:2450AT18D0100E
- added J12: A3-16DA-2SV(71), 16pos2mm1:A3-16DA-2SV(71), symbol 16pos_2mm_SMD:A3-16DA-2SV(71)
- added J13: 0877601616, 16pos2mmRA:62401621722, symbol 16pos2mmRA:0877601616
- added M1: Pos-1a, gsg-modules:TESTPOINT-50MIL, symbol Connector:TestPoint
- added M2: Neg-1a, gsg-modules:TESTPOINT-50MIL, symbol Connector:TestPoint
- added M3: Pos-2a, gsg-modules:TESTPOINT-50MIL, symbol Connector:TestPoint
- added M4: Neg-2a, gsg-modules:TESTPOINT-50MIL, symbol Connector:TestPoint
- P1: footprint (none) -> library:SWD_6pin
- P4: footprint (none) -> Connector_DIN:Conn_01x02_Female
- P5: footprint (none) -> library:ExternalPort
Connections:
- net labels removed: 10a_SDA, 11a_SCL, 15a_GND2, 15b_GND2, 21b_3.3v, 23b_GND, 8a_IO1, 9a_IO2, GND
- wire segments 374 -> 418
- no-connect marks 35 -> 27

Commit message: Routed PCBs pending optimization
Parts:
- J12: footprint 16pos2mm1:A3-16DA-2SV(71) -> A13:A13_1; symbol 16pos_2mm_SMD:A3-16DA-2SV(71) -> 16pos2mmRA:0877601616
Connections:
- net labels added: 23a_Ground
- net labels removed: 23a_GND, NSRT
- wire segments 418 -> 408
- no-connect marks 27 -> 52

Commit message: Updated copper cores; changed schematic naming flags for 3rd party BOM generator; added renders of board; added some datasheets
Parts:
- removed M1: Pos-1a, gsg-modules:TESTPOINT-50MIL, symbol Connector:TestPoint
- removed M2: Neg-1a, gsg-modules:TESTPOINT-50MIL, symbol Connector:TestPoint
- removed M3: Pos-2a, gsg-modules:TESTPOINT-50MIL, symbol Connector:TestPoint
- removed M4: Neg-2a, gsg-modules:TESTPOINT-50MIL, symbol Connector:TestPoint
- removed P1: SWD Pads, library:SWD_6pin, symbol Connector_Generic:Conn_01x06
- removed P4: Conn_01x02_Female, Connector_DIN:Conn_01x02_Female, symbol Connector:Conn_01x02_Female
- removed P5: Pads, library:ExternalPort, symbol Connector:Conn_01x06_Female
- removed R25, R26: NC, footprints:ERJ-2GE0R00X, symbol Device:R_US
- A1: renamed from ANT1; manf# (none) -> 2450AT18D0100E; mnf# (none) -> 2450AT18D0100E
- B1: manf# (none) -> 2450BM14A0002T; mnf# (none) -> 2450BM14A0002T
- C1: manf# (none) -> C0402C103J3RACTU; mnf# (none) -> C0402C103J3RACTU
- C10, C11, C14, C17, C18, C4, C5, C6: manf# (none) -> LMK107BJ475KA-T; mnf# (none) -> LMK107BJ475KAT
- C12, C13, C2: manf# (none) -> 0603ZD105KAT2A; mnf# (none) -> 0603ZD105KAT2A
- C15, C16, C3: manf# (none) -> CL10A475KP8NNNC; mnf# (none) -> CL10A475KP8NNNC
- C19: value 100nF -> 10nF; footprint 100nf:C0402C104K4RACTU -> 10nF:C0402C103J3RACTU; manf# (none) -> C0402C103J3RACTU; mnf# (none) -> C0402C103J3RACTU
- C20: value 100nF -> 1nF; manf# (none) -> C0402C102K5RACTU; mnf# (none) -> C0402C102K5RACTU
- C21: manf# (none) -> C0402C222K5RACTU; mnf# (none) -> C0402C222K5RACTU
- C22: manf# (none) -> CGA2B3X7R1H333K050BB; mnf# (none) -> CGA2B3X7R1H333K050BB
- C7, C8: manf# (none) -> GRM1555C1H220JA01D; mnf# (none) -> GRM1555C1H220JA01D
- C9: manf# (none) -> GRM188R61A106ME9D; mnf# (none) -> GRM188R61A106ME9D
- D1, D3: manf# (none) -> PD15-22C/TR8; mnf# (none) -> PD1522CTR8
- D2: manf# (none) -> SMLVN6RGB1W1; mnf# (none) -> SMLVN6RGB1W1
- J1: value MOLEX_78171-0002 -> MOLEX781710002; manf# (none) -> 78171-0002; mnf# (none) -> 781710002
- J10, J12: value A3-16DA-2SV(71) -> A316DA2SV71; manf# (none) -> A3-16DA-2SV(71); mnf# (none) -> A316DA2SV71
- J11: manf# (none) -> 0877601616; mnf# (none) -> 0877601616
- J13: manf# (none) -> 0877581616; mnf# (none) -> 0877581616
- J2: value MOLEX_78171-0003 -> MOLEX781710003; manf# (none) -> 78171-0003; mnf# (none) -> 781710003
- Q1, Q2, Q3, Q4: manf# (none) -> MMBT3904LT1G; mnf# (none) -> MMBT3904LT1G
- R1, R2, R3: manf# (none) -> MCMR04X22R0FTL; mnf# (none) -> MCMR04X22R0FTL
- R10, R13: manf# (none) -> RC0402FR-07560KL; mnf# (none) -> RC0402FR-07560KL
- R11, R21: manf# (none) -> CRCW04021M50FKED; mnf# (none) -> CRCW04021M50FKED
- R12, R15, R23, R4, R5, R6, R8: manf# (none) -> CRCW0402100KFKED; mnf# (none) -> CRCW0402100KFKED
- R14, R19, R20, R22, R7, R9: manf# (none) -> CRCW040210K0FKED; mnf# (none) -> CRCW040210K0FKED
- R16: manf# (none) -> ERJ-2RKF22R6X; mnf# (none) -> ERJ2RKF22R6X
- R17: manf# (none) -> RVC0402FT130K; mnf# (none) -> RVC0402FT130K
- R18: manf# (none) -> ERJ-2RKF24R9X; mnf# (none) -> ERJ2RKF24R9X
- R24: manf# (none) -> RC0402JR-070RL; mnf# (none) -> RC0402JR070RL
- R27: manf# (none) -> CRCW040222K0FKED; mnf# (none) -> CRCW040222K0FKED
- U1: manf# (none) -> STM32F051C8U6; mnf# (none) -> STM32F051C8U6
- U2: DK_Datasheet_Link (none) -> https://www.st.com/content/ccc/resource/technical/document/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; manf# (none) -> LSM6DS3TR; mnf# (none) -> LSM6DS3TR
- U3: value A3901SEJTR-T -> A3901SEJTRT; manf# (none) -> A3901SEJTR-T; mnf# (none) -> A3901SEJTRT
- U4: value ADP122ACPZ-3.3-R7 -> ADP122ACPZ33R7; manf# (none) -> ADP122ACPZ-3.3-R7; mnf# (none) -> ADP122ACPZ33R7
- U5: value AT42QT1070-MMHCT-ND -> AT42QT1070MMHCTND; manf# (none) -> AT42QT1070-MMHR; mnf# (none) -> AT42QT1070MMHR
- U6: value MCP73831T-2ACI_OT -> MCP73831T2ACIOT; manf# (none) -> MCP73831T-2ACI/OT; mnf# (none) -> MCP73831T2ACIOT
- U7: value NRF24L01P-R7 -> NRF24L01PR7; manf# (none) -> NRF24L01P-R7; mnf# (none) -> NRF24L01PR7
- Y1: value 7V-16.000MAAE-T -> 7V16000MAAET; manf# (none) -> 7V-16.000MAAE-T; mnf# (none) -> 7V16000MAAET
Connections:
- net labels added: 10bSDA, 11bSCL, 12aA1, 12bA1, 13aA2, 13bA2, 14aVDDPA, 14bVDDPA, 15aP41, 15bP41, 1a33v, 1b33v, 21a3.3v, 21a33v, 22aVBAT, 22bVBAT, 23aGround, 24aIMUINT, 24bIMUINT, 25aSDA, 25bSDA, 26aSCL, 26bSCL, 27aCHARGING, 27bCHARGING, 28aP41, 2aGND, 2bGND, 3aPHOTODIODE1, 3bPHOTODIODE1, 4aPHOTODIODE2, 4bPHOTODIODE2, 5aRGBLED1, 5bRGBLED1, 6aRGBLED2, 6bRGBLED2, 7aRGBLED3, 7bRGBLED3, 8bIO1, 9bIO2, MCUX116MHZ, MCUX216MHZ, MOTORCONTROL1, MOTORCONTROL2, MOTORCONTROL3, MOTORCONTROL4, RADIOCLK, RADIOIRQ, ~29aTOUCHCHG~, ~29bTOUCHCHG~
- net labels removed: 10b_SDA, 11b_SCL, 12a_ANT1, 12b_ANT1, 13a_ANT2, 13b_ANT2, 14a_VDD_PA, 14b_VDD_PA, 15a_P4-1, 15b_P4-1, 1a_3.3v, 1b_3.3v, 21a_3.3v, 22a_VBAT, 22b_VBAT, 24a_IMU_INT, 24b_IMU_INT, 25a_SDA, 25b_SDA, 26a_SCL, 26b_SCL, 27a_CHARGING, 27b_CHARGING, 28a_P4-1, 2a_GND, 2b_GND, 3a_PHOTODIODE1, 3b_PHOTODIODE1, 4a_PHOTODIODE2, 4b_PHOTODIODE2, 5a_RGBLED1, 5b_RGBLED1, 6a_RGBLED2, 6b_RGBLED2, 7a_RGBLED3, 7b_RGBLED3, 8b_IO1, 9b_IO2, MCU_X1_16MHZ, MCU_X2_16MHZ, MOTOR_CONTROL1, MOTOR_CONTROL2, MOTOR_CONTROL3, MOTOR_CONTROL4, RADIO_IRQ, ~29a_TOUCH_CHG~, ~29b_TOUCH_CHG~
