File: SKINNY_PROTOTYPE/BB_Hardware/PCB/BadukBot/BotSchematic/BotSchematic.sch (KiCad schematic (older format))
At the start: 70 parts, among them J1 MOLEX781710002, J10 A316DA2SV71, J11 62401621722, J12 A316DA2SV71, J13 0877601616, J2 MOLEX781710003, Q1 MMBT3904LT1G, Q2 MMBT3904LT1G, Q3 MMBT3904LT1G, Q4 MMBT3904LT1G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

Commit message: Added images of the board; minor changes to BOM; Attempts to use KiCost to automate component shopping; Minor changes to copper pours on board
Working on getting KiCost to work with the xml generated by KiCAD to make shopping for parts easy at Octopart. Looks to be approx $20 per board
Parts:
- C9: manf# GRM188R61A106ME9D -> GRM188R61A106ME69D; mnf# GRM188R61A106ME9D -> GRM188R61A106ME69D
Connections:
- wire segments 408 -> 405
Changed lines of the file:
@@
 Wire Wire Line
 	15850 1550 15900 1550
-Wire Wire Line
-	15900 1600 15900 1550
 Connection ~ 15900 1550
-Wire Wire Line
-	15300 1600 15300 1550
 Wire Wire Line
 	15300 1550 15350 1550
@@
 F 2 "10uF:CAPC1608X9N" H 14350 5200 50  0001 L BNN
 F 3 "0603 Murata" H 14350 5200 50  0001 L BNN
-F 4 "Multilayer Ceramic Capacitor, GRM Series, 10 F, 20%, X5R, 10 V, 0603 [1608 Metric]" H 14350 5200 50  0001 L BNN "Field4"
-F 5 "GRM188R61A106ME69D" H 14350 5200 50  0001 L BNN "Field5"
-F 6 "None" H 14350 5200 50  0001 L BNN "Field6"
-F 7 "Murata" H 14350 5200 50  0001 L BNN "Field7"
-F 8 "Unavailable" H 14350 5200 50  0001 L BNN "Field8"
-F 9 "GRM188R61A106ME9D" H 0   0   50  0001 C CNN "mnf#"
-F 10 "GRM188R61A106ME9D" H 0   0   50  0001 C CNN "manf#"
+F 4 "GRM188R61A106ME69D" H 0   0   50  0001 C CNN "manf#"
+F 5 "Multilayer Ceramic Capacitor, GRM Series, 10 F, 20%, X5R, 10 V, 0603 [1608 Metric]" H 14350 5200 50  0001 L BNN "Field4"
+F 6 "GRM188R61A106ME69D" H 14350 5200 50  0001 L BNN "Field5"
+F 7 "None" H 14350 5200 50  0001 L BNN "Field6"
+F 8 "Murata" H 14350 5200 50  0001 L BNN "Field7"
+F 9 "Unavailable" H 14350 5200 50  0001 L BNN "Field8"
+F 10 "GRM188R61A106ME69D" H 0   0   50  0001 C CNN "mnf#"
 	1    14350 5200
 	0    -1   -1   0
@@
 Wire Wire Line
 	14900 2250 14850 2250
-Wire Wire Line
-	15300 1900 15300 2550
 $Comp
 L 16pos_2mm_SMD:A3-16DA-2SV(71) J10
@@
 	12300 5150 12300 5550
 Wire Wire Line
-	14750 1850 14700 1850
-Connection ~ 14700 1850
-Wire Wire Line
 	8000 2650 8000 2700
 Wire Wire Line
@@
 Wire Wire Line
 	16500 2650 15900 2650
-Wire Wire Line
-	15900 1900 15900 2650
 Text GLabel 15050 1250 2    50   BiDi ~ 0
 2aGND
@@
 Text GLabel 13350 6050 2    50   BiDi ~ 0
 21a33v
+Wire Wire Line
+	15300 1550 15300 2550
+Wire Wire Line
+	15900 1550 15900 2650
 $EndSCHEMATC
