File: SKINNY_PROTOTYPE/BB_Hardware/PCB/BadukBot/BotSchematic/_autosave-BotSchematicRouted_v03.kicad_pcb (KiCad board)
At the start: 2 copper layers, 93.5 x 43.6 mm, 118 parts, among them J1 MOLEX781710002, J10 A316DA2SV71, J11 62401621722, J12 A316DA2SV71, J13 0877601616, J2 MOLEX781710003, M1 Pos1a, M2 Neg1a, M3 Pos2a, M4 Neg2a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

Commit message: Changed PCB for more compact component placement, shortened board 3, added images for the new layout
Parts:
- moved G2 7.06 mm to (132.2, 87.5)
- moved G1 7.06 mm to (142.1, 80.2)
- renumbered P4 to P10
Routing:
- net 23aGround: track 123.9 -> 127.2 mm, vias 29 -> 31
- net 4aPHOTODIODE2: track 22.8 -> 24.0 mm
- net 1a33v: track 62.0 -> 63.0 mm, vias 8 -> 10
- net 2bGND: vias 29 -> 31
