File: SKINNY_PROTOTYPE/BB_Hardware/PCB/BadukBot/BotSchematic/BotSchematicRouted_v03.kicad_pcb (KiCad board)
At the start: 2 copper layers, 73 x 22.5 mm, 89 parts, among them J1 MOLEX781710002, J10 A316DA2SV71, J11 62401621722, J12 A316DA2SV71, J13 62401621722, J2 MOLEX781710003, M1 Pos1a, M2 Neg1a, M3 Pos2a, M4 Neg2a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

Commit message: PCB revisions
Parts:
- added P4: Conn_01x02_Female, Connector_DIN:Conn_01x02_Female, B.Cu at (84.1, 104.6)
- moved G2 7.56 mm to (77.5, 105.2)
- moved G1 6.83 mm to (84.7, 105.2)
- moved G5 1.61 mm to (83.6, 111.8)
Changed lines of the file:
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@@
   (general
     (thickness 1.6)
-    (drawings 252)
-    (tracks 2291)
+    (drawings 250)
+    (tracks 2292)
     (zones 0)
-    (modules 89)
+    (modules 90)
     (nets 137)
   )
@@
   )
   (module Silk:OpenHardwareLogo (layer B.Cu)
-    (at 85.06 104.38 90)
+    (at 77.54 105.19 90)
     (fp_text reference G2 (at 0 0 90) (layer B.SilkS) hide
       (effects (font (size 1.524 1.524) (thickness 0.3)) (justify mirror))
@@
   )
   (module Silk:BadukBot-GoSwarm (layer B.Cu)
-    (at 77.89 104.64 90)
+    (at 84.7 105.2 90)
     (fp_text reference G1 (at 0 0 90) (layer B.SilkS) hide
       (effects (font (size 1.524 1.524) (thickness 0.3)) (justify mirror))
@@
   )
   (module Silk:links_20mm (layer B.Cu)
-    (at 83.66 110.14)
+    (at 83.58 111.75)
     (fp_text reference G5 (at 0 0) (layer B.SilkS) hide
       (effects (font (size 1.524 1.524) (thickness 0.3)) (justify mirror))
@@
     (pad 2 smd circle (at 1.1 0 315) (size 1.524 1.524) (layers B.Cu B.Paste B.Mask))
   )
+  (module Connector_DIN:Conn_01x02_Female (layer B.Cu)
+    (at 84.1 104.58 315)
+    (attr smd)
+    (fp_text reference P4 (at 0 -1.5 315) (layer B.SilkS) hide
+      (effects (font (size 1 1) (thickness 0.15)) (justify mirror))
+    )
+    (fp_text value Conn_01x02_Female (at 0 1.15 315) (layer B.SilkS) hide
+      (effects (font (size 0.5 0.5) (thickness 0.125)) (justify mirror))
+    )
+    (pad 1 smd circle (at -1.15 0 315) (size 1.524 1.524) (layers B.Cu B.Paste B.Mask))
+    (pad 2 smd circle (at 1.1 0 315) (size 1.524 1.524) (layers B.Cu B.Paste B.Mask))
+  )
   (gr_line (start 129.63 100.1) (end 129.63 115.5) (layer F.SilkS) (width 0.2))
   (gr_line (start 144.17 100.09) (end 144.17 115.49) (layer F.SilkS) (width 0.2))
@@
   (gr_line (start 137.45 100.08) (end 141.84 100.08) (layer B.SilkS) (width 0.2))
   (gr_line (start 137.45 115.51) (end 141.84 115.51) (layer B.SilkS) (width 0.2))
-  (gr_line (start 110.97 115.43) (end 115.36 115.41) (layer B.SilkS) (width 0.2))
-  (gr_line (start 110.97 99.94) (end 115.36 99.92) (layer B.SilkS) (width 0.2))
-  (gr_line (start 115.36 99.92) (end 115.36 115.41) (layer B.SilkS) (width 0.2))
-  (gr_line (start 110.97 99.94) (end 110.97 115.43) (layer B.SilkS) (width 0.2))
+  (gr_line (start 110.97 115.59) (end 115.36 115.59) (layer B.SilkS) (width 0.2))
+  (gr_line (start 110.97 99.94) (end 115.36 99.94) (layer B.SilkS) (width 0.2))
+  (gr_line (start 115.36 99.94) (end 115.36 115.59) (layer B.SilkS) (width 0.2))
+  (gr_line (start 110.97 99.94) (end 110.97 115.59) (layer B.SilkS) (width 0.2))
   (gr_line (start 93.9 100.01) (end 93.9 115.5) (layer B.SilkS) (width 0.2))
   (gr_line (start 103.42 100.02) (end 103.42 115.51) (layer B.SilkS) (width 0.2))
@@
   (gr_line (start 93.9 100) (end 93.9 111.78) (layer F.SilkS) (width 0.2))
   (gr_line (start 87.39 114.79) (end 87.85 113.75) (layer F.SilkS) (width 0.2))
-  (gr_circle (center 78.06 104.79) (end 78.05 105.51) (layer B.SilkS) (width 0.2))
-  (gr_circle (center 76.48 103.22) (end 76.47 103.94) (layer B.SilkS) (width 0.2))
   (gr_line (start 120.23 115.02) (end 119.97 115.02) (layer F.SilkS) (width 0.2))
   (gr_line (start 120.23 114.56) (end 120.23 115.02) (layer F.SilkS) (width 0.2))
@@
   (segment (start 119.37868 101.809148) (end 120.12868 102.559148) (width 0.1524) (layer F.Cu) (net 89))
   (segment (start 120.12868 102.559148) (end 122.42868 102.559148) (width 0.1524) (layer F.Cu) (net 89) (status 20))
-  (segment (start 116.27868 102.9) (end 116.27868 107.759148) (width 0.1524) (layer F.Cu) (net 89) (status 20))
-  (segment (start 117 102.9) (end 117.27 102.63) (width 0.1524) (layer F.Cu) (net 89))
-  (segment (start 116.27868 102.9) (end 117 102.9) (width 0.1524) (layer F.Cu) (net 89))
   (segment (start 114.715736 108.88) (end 115.14 108.88) (width 0.1524) (layer F.Cu) (net 89))
   (segment (start 114.62 108.975736) (end 114.715736 108.88) (width 0.1524) (layer F.Cu) (net 89))
@@
   (segment (start 111.705032 102.428948) (end 110.851073 102.428948) (width 0.25) (layer F.Cu) (net 90))
   (segment (start 113.55768 103.509148) (end 113.55768 103.688753) (width 0.25) (layer F.Cu) (net 90))
-  (segment (start 116.87868 103.509148) (end 116.87868 104.659148) (width 0.25) (layer B.Cu) (net 90))
   (via (at 119.21 107.24) (size 0.6) (drill 0.3) (layers F.Cu B.Cu) (net 90))
   (segment (start 119.109532 107.139532) (end 119.21 107.24) (width 0.1524) (layer B.Cu) (net 90))
@@
   (segment (start 119.27 107.29) (end 119.569999 107.589999) (width 0.25) (layer F.Cu) (net 90))
   (via (at 113.55768 103.509148) (size 0.6) (drill 0.3) (layers F.Cu B.Cu) (net 90))
-  (segment (start 116.87868 103.509148) (end 113.55768 103.509148) (width 0.25) (layer B.Cu) (net 90))
   (via (at 110.851073 102.750972) (size 0.6) (drill 0.3) (layers F.Cu B.Cu) (net 90) (status 30))
   (segment (start 110.851073 102.750972) (end 110.851073 102.428948) (width 0.1524) (layer F.Cu) (net 90))
@@
   (segment (start 115.483258 105.485557) (end 115.451073 105.453372) (width 0.1524) (layer B.Cu) (net 84))
   (segment (start 116.924443 105.485557) (end 115.483258 105.485557) (width 0.1524) (layer B.Cu) (net 84))
+  (segment (start 116.27868 103.62132) (end 117.27 102.63) (width 0.1524) (layer F.Cu) (net 89))
+  (segment (start 116.27868 107.759148) (end 116.27868 103.62132) (width 0.1524) (layer F.Cu) (net 89))
+  (segment (start 116.307828 103.509148) (end 116.87868 104.08) (width 0.25) (layer B.Cu) (net 90))
+  (segment (start 115.56 103.509148) (end 116.307828 103.509148) (width 0.25) (layer B.Cu) (net 90))
+  (segment (start 115.56 103.509148) (end 113.55768 103.509148) (width 0.25) (layer B.Cu) (net 90))
+  (segment (start 116.87868 104.08) (end 116.87868 104.659148) (width 0.25) (layer B.Cu) (net 90))
   (segment (start 103.840849 100.926367) (end 103.605185 100.690703) (width 0.1524) (layer F.Cu) (net 93))
   (segment (start 103.840849 110.395637) (end 103.840849 100.926367) (width 0.1524) (layer F.Cu) (net 93))
